File: clock_timer.kicad_sch (KiCad schematic)
At the start: 11 parts, among them SW1 SW_Push, U1 LM555xN, U2 LM555xN, U3 LM555xN

Commit message: Add files via upload
Parts:
- added C4: C, symbol Device:C
- added D1: LED, symbol Device:LED
- added R5, R6, R7: R, symbol Device:R
- added SW2: SW_SPDT, symbol Switch:SW_SPDT
- added U4: 74LS04, symbol 74xx:74LS04
- added U5: 74LS32, symbol 74xx:74LS32
- added U6: 74LS08, symbol 74xx:74LS08
Connections:
- net +5V: now also U3.8 (VCC), R5.1, R6.1
- net GND: now also U3.1 (GND), U3.6 (THR), C4.2, D1.1 (K), SW2.2 (B), U4.3
- net at U3.2 (TR): now also R6.2, SW2.1 (A)
- net at U3.3 (Q): now also U4.1, U6.2
- net at U3.4 (R): now also U3.5 (CV), C4.1, R5.2, SW2.3 (C)
- net at U2.3 (Q): now also U6.5
- net at R1.2, R2.1, U1.7 (DIS): no longer U1.3 (Q)
- new net: R7.1, U6.8
- new net: D1.2 (A), R7.2
- new net: U5.1, U6.3
- new net: U5.2, U6.6
- new net: U5.3, U6.9
- new net: U1.3 (Q), U6.1
- new net: U4.2, U6.4
- new net: U4.4, U6.10
